Commit message: add cube wight

File: python/pybullet/grasping_demo/dish/box.urdf (robot description, URDF)
Before this commit: robot block_2, 1 links, 0 joints
Links:
- link block_2_base_link: mass 0.2 -> 1000

Commit message: edit cube inertia, mass, size

File: python/pybullet/grasping_demo/dish/box.urdf (robot description, URDF)
Before this commit: robot block_2, 1 links, 0 joints
Links:
- link block_2_base_link: mass 1000 -> 10000; geometry collision box size=0.6 1.9 0.55; visual box size=0.6 1.65 0.55
